File: fwr/fwr.kicad_pcb (KiCad board)
At the start: 2 copper layers, 49 x 99 mm, 35 parts, among them J1 CV_Input, J2 Input, J3 Synth_power_2x5, J4 Output, U1 TL074

Commit message: buncha
Parts:
- removed Bias1, CV_Amount1, Feedback1: 100K, ao_tht:Molex_KK-254_AE-6410-03A_1x03_P2.54mm_Vertical
- removed D1, D2: 1N4148, Diode_THT:D_DO-35_SOD27_P7.62mm_Horizontal
- removed D3, D4: 1N4733, Diode_THT:D_DO-41_SOD81_P10.16mm_Horizontal
- added  : MountingHole, ao_tht:MountingHole_3.2mm_M3, F.Cu at (143.5, 143.0)
- added 1N4148: 1N4148, Diode_THT:D_DO-35_SOD27_P7.62mm_Horizontal, F.Cu at (127.5, 137.5)
- added 1N4148: 1N4148, Diode_THT:D_DO-35_SOD27_P7.62mm_Horizontal, F.Cu at (116.0, 137.5)
- added 1N4733: 1N4733, Diode_THT:D_DO-41_SOD81_P10.16mm_Horizontal, F.Cu at (118.5, 65.0)
- added 1N4733: 1N4733, Diode_THT:D_DO-41_SOD81_P10.16mm_Horizontal, F.Cu at (118.5, 70.0)
- added Bias: 100K, ao_tht:Molex_KK-254_AE-6410-03A_1x03_P2.54mm_Vertical, B.Cu at (106.5, 56.0)
- added CV_Amount: 100K, ao_tht:Molex_KK-254_AE-6410-03A_1x03_P2.54mm_Vertical, B.Cu at (121.0, 56.0)
- added Feedback: 100K, ao_tht:Molex_KK-254_AE-6410-03A_1x03_P2.54mm_Vertical, B.Cu at (135.5, 56.0)
- moved R13 44.2 mm to (105.0, 95.5)
- moved R9 42.6 mm to (105.0, 77.5)
- moved R1 39.7 mm to (135.5, 86.5)
- moved H1 39.1 mm to (145.5, 54.0)
- moved R14 33.4 mm to (105.0, 82.0)
- moved FB1 33.2 mm to (124.5, 115.0)
- moved U1 31.9 mm to (105.0, 106.0)
- moved R8 28.6 mm to (120.5, 77.6)
- moved J1 26.7 mm to (108.0, 66.5)
- moved R5 26.0 mm to (127.5, 132.5)
- moved C3 23.2 mm to (118.5, 123.0)
- moved R4 22.8 mm to (120.3, 90.1)
- moved R12 21.1 mm to (135.5, 91.0)
- moved R7 20.3 mm to (120.5, 81.6)
- moved C5 18.6 mm to (129.5, 124.0)
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Routing:
- net -12V: track 0.00 -> 225.8 mm
- net Net-(Feedback1-Pad3): track 0.00 -> 129.0 mm
- net +12V: track 0.00 -> 125.6 mm
- net Net-(D3-Pad2): track 0.00 -> 108.1 mm
- net Net-(D1-Pad2): track 0.00 -> 81.3 mm
- net Net-(R5-Pad1): track 0.00 -> 77.6 mm
- net Net-(C4-Pad2): track 0.00 -> 74.0 mm
- net Net-(R12-Pad1): track 0.00 -> 70.9 mm
- net Net-(R2-Pad1): track 0.00 -> 50.8 mm
- net Net-(CV_Amount1-Pad2): track 0.00 -> 50.5 mm
- net Net-(R6-Pad2): track 0.00 -> 49.7 mm
- net Net-(C1-Pad2): track 0.00 -> 48.7 mm
- net Net-(Bias1-Pad2): track 0.00 -> 44.4 mm
- net Net-(D2-Pad1): track 0.00 -> 32.0 mm
- net Net-(D1-Pad1): track 0.00 -> 29.2 mm
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Other:
- board text added: "FWR! Rich Jones! LMNC Golf 2021!"
- board text added: "Full Wave Rectifier!"
