File: fwr/fwr.sch (KiCad schematic (older format))
At the start: 35 parts, among them J1 CV_Input, J2 Input, J3 Synth_power_2x5, J4 Output, U1 TL074

Commit message: buncha
Parts:
- added H2: MountingHole, MountingHole:MountingHole_3.2mm_M3, symbol Mechanical:MountingHole
- C5, C6: value C_Polarized -> 10uf
- J2: footprint ao_tht:Molex_KK-254_AE-6410-03A_1x03_P2.54mm_Vertical -> ao_tht:Molex_KK-254_AE-6410-02A_1x02_P2.54mm_Vertical
Changed lines of the file:
@@
 F 0 "J2" H 2568 2442 50  0000 C CNN
 F 1 "Input" H 2568 2351 50  0000 C CNN
-F 2 "ao_tht:Molex_KK-254_AE-6410-03A_1x03_P2.54mm_Vertical" H 2650 2225 50  0001 C CNN
+F 2 "ao_tht:Molex_KK-254_AE-6410-02A_1x02_P2.54mm_Vertical" H 2650 2225 50  0001 C CNN
 F 3 "" H 2650 2225 50  0001 C CNN
 	1    2650 2225
@@
 F 1 "Synth_power_2x5" H 5575 5691 60  0000 C CNN
 F 2 "ao_tht:Power_Header" H 5575 5350 60  0001 C CNN
-F 3 "" H 5575 5350 60  0000 C CNN
+F 3 "" H 5575 5350 60  0001 C CNN
 	1    5575 5350
 	1    0    0    -1
@@
 L power:GND #PWR017
 U 1 1 60ED1FF2
-P 7100 5350
-F 0 "#PWR017" H 7100 5100 50  0001 C CNN
-F 1 "GND" H 7105 5177 50  0000 C CNN
-F 2 "" H 7100 5350 50  0001 C CNN
-F 3 "" H 7100 5350 50  0001 C CNN
-	1    7100 5350
+P 7100 5600
+F 0 "#PWR017" H 7100 5350 50  0001 C CNN
+F 1 "GND" H 7105 5427 50  0000 C CNN
+F 2 "" H 7100 5600 50  0001 C CNN
+F 3 "" H 7100 5600 50  0001 C CNN
+	1    7100 5600
 	1    0    0    -1
 $EndComp
@@
 P 6800 5750
 F 0 "C6" H 6918 5796 50  0000 L CNN
-F 1 "C_Polarized" H 6918 5705 50  0000 L CNN
+F 1 "10uf" H 6918 5705 50  0000 L CNN
 F 2 "ao_tht:CP_Radial_D5.0mm_P2.00mm" H 6838 5600 50  0001 C CNN
 F 3 "~" H 6800 5750 50  0001 C CNN
@@
 P 6800 5075
 F 0 "C5" H 6918 5121 50  0000 L CNN
-F 1 "C_Polarized" H 6918 5030 50  0000 L CNN
+F 1 "10uf" H 6918 5030 50  0000 L CNN
 F 2 "ao_tht:CP_Radial_D5.0mm_P2.00mm" H 6838 4925 50  0001 C CNN
 F 3 "~" H 6800 5075 50  0001 C CNN
@@
 Connection ~ 6800 5900
 Wire Wire Line
-	7100 5350 6800 5350
-Wire Wire Line
-	6800 5600 6800 5350
+	7100 5600 6800 5600
 Connection ~ 6800 5600
-Connection ~ 6800 5350
-Wire Wire Line
-	6800 5350 6025 5350
-Wire Wire Line
-	6800 5225 6800 5350
 Wire Wire Line
 	6600 5025 6600 4925
@@
 Wire Wire Line
 	6025 5025 6025 4775
-Wire Wire Line
-	6025 4775 5600 4775
 Wire Wire Line
 	5125 4775 5125 5150
@@
 	3700 5950 3700 6075
 Wire Wire Line
-	3700 5825 3700 5850
-Connection ~ 3700 5850
-Wire Wire Line
 	3700 5850 3700 5950
 Wire Wire Line
@@
 Wire Wire Line
 	6800 3775 6800 3800
-$Comp
-L power:PWR_FLAG #FLG0101
-U 1 1 60FFCF37
-P 5600 4700
-F 0 "#FLG0101" H 5600 4775 50  0001 C CNN
-F 1 "PWR_FLAG" H 5600 4873 50  0000 C CNN
-F 2 "" H 5600 4700 50  0001 C CNN
-F 3 "~" H 5600 4700 50  0001 C CNN
-	1    5600 4700
-	1    0    0    -1
-$EndComp
-Wire Wire Line
-	5600 4700 5600 4775
-Connection ~ 5600 4775
-Wire Wire Line
-	5600 4775 5125 4775
-$Comp
-L power:PWR_FLAG #FLG0102
-U 1 1 610018C0
-P 4950 5250
-F 0 "#FLG0102" H 4950 5325 50  0001 C CNN
-F 1 "PWR_FLAG" H 4950 5423 50  0000 C CNN
-F 2 "" H 4950 5250 50  0001 C CNN
-F 3 "~" H 4950 5250 50  0001 C CNN
-	1    4950 5250
-	1    0    0    -1
-$EndComp
-$Comp
-L power:PWR_FLAG #FLG0103
-U 1 1 61005AE0
-P 5575 5825
-F 0 "#FLG0103" H 5575 5900 50  0001 C CNN
-F 1 "PWR_FLAG" H 5575 5998 50  0000 C CNN
-F 2 "" H 5575 5825 50  0001 C CNN
-F 3 "~" H 5575 5825 50  0001 C CNN
-	1    5575 5825
-	1    0    0    1
-$EndComp
-Wire Wire Line
-	5125 5825 5575 5825
-Connection ~ 5575 5825
-Wire Wire Line
-	5575 5825 6025 5825
-Wire Wire Line
-	5125 5350 4950 5350
-Wire Wire Line
-	4950 5250 4950 5350
-Connection ~ 4950 5350
-Wire Wire Line
-	4950 5350 4850 5350
 $Comp
 L power:+12V #PWR0101
@@
 $EndComp
 Wire Wire Line
-	3700 4850 3700 5150
+	3700 4850 3700 5050
 Connection ~ 3700 5150
 Wire Wire Line
@@
 	1    0    0    -1
 $EndComp
+$Comp
+L Mechanical:MountingHole H2
+U 1 1 611578CE
+P 1850 5475
+F 0 "H2" H 1950 5521 50  0000 L CNN
+F 1 "MountingHole" H 1950 5430 50  0000 L CNN
+F 2 "MountingHole:MountingHole_3.2mm_M3" H 1850 5475 50  0001 C CNN
+F 3 "~" H 1850 5475 50  0001 C CNN
+	1    1850 5475
+	1    0    0    -1
+$EndComp
+Wire Wire Line
+	5125 5825 5625 5825
+Wire Wire Line
+	5125 4775 5625 4775
+$Comp
+L power:GND #PWR0104
+U 1 1 612E5FF2
+P 6300 5350
+F 0 "#PWR0104" H 6300 5100 50  0001 C CNN
+F 1 "GND" H 6305 5177 50  0000 C CNN
+F 2 "" H 6300 5350 50  0001 C CNN
+F 3 "" H 6300 5350 50  0001 C CNN
+	1    6300 5350
+	1    0    0    -1
+$EndComp
+Wire Wire Line
+	6025 5350 6300 5350
+$Comp
+L power:PWR_FLAG #FLG0102
+U 1 1 6130B3EB
+P 5625 4750
+F 0 "#FLG0102" H 5625 4825 50  0001 C CNN
+F 1 "PWR_FLAG" H 5625 4923 50  0000 C CNN
+F 2 "" H 5625 4750 50  0001 C CNN
+F 3 "~" H 5625 4750 50  0001 C CNN
+	1    5625 4750
+	1    0    0    -1
+$EndComp
+$Comp
+L power:PWR_FLAG #FLG0103
+U 1 1 6130F65E
+P 5625 5800
+F 0 "#FLG0103" H 5625 5875 50  0001 C CNN
+F 1 "PWR_FLAG" H 5625 5973 50  0000 C CNN
+F 2 "" H 5625 5800 50  0001 C CNN
+F 3 "~" H 5625 5800 50  0001 C CNN
+	1    5625 5800
+	1    0    0    -1
+$EndComp
+Wire Wire Line
+	5625 4750 5625 4775
+Connection ~ 5625 4775
+Wire Wire Line
+	5625 4775 6025 4775
+Wire Wire Line
+	5625 5800 5625 5825
+Connection ~ 5625 5825
+Wire Wire Line
+	5625 5825 6025 5825
+$Comp
+L power:PWR_FLAG #FLG0104
+U 1 1 613338C4
+P 3700 5050
+F 0 "#FLG0104" H 3700 5125 50  0001 C CNN
+F 1 "PWR_FLAG" V 3700 5177 50  0000 L CNN
+F 2 "" H 3700 5050 50  0001 C CNN
+F 3 "~" H 3700 5050 50  0001 C CNN
+	1    3700 5050
+	0    -1   -1   0
+$EndComp
+Connection ~ 3700 5050
+Wire Wire Line
+	3700 5050 3700 5150
+Wire Wire Line
+	4850 5350 4975 5350
+$Comp
+L power:PWR_FLAG #FLG0101
+U 1 1 61358670
+P 4975 5300
+F 0 "#FLG0101" H 4975 5375 50  0001 C CNN
+F 1 "PWR_FLAG" H 4975 5473 50  0000 C CNN
+F 2 "" H 4975 5300 50  0001 C CNN
+F 3 "~" H 4975 5300 50  0001 C CNN
+	1    4975 5300
+	1    0    0    -1
+$EndComp
+Wire Wire Line
+	4975 5300 4975 5350
+Connection ~ 4975 5350
+Wire Wire Line
+	4975 5350 5125 5350
+$Comp
+L power:GND #PWR0105
+U 1 1 6136B6BB
+P 7100 5300
+F 0 "#PWR0105" H 7100 5050 50  0001 C CNN
+F 1 "GND" H 7105 5127 50  0000 C CNN
+F 2 "" H 7100 5300 50  0001 C CNN
+F 3 "" H 7100 5300 50  0001 C CNN
+	1    7100 5300
+	1    0    0    -1
+$EndComp
+Wire Wire Line
+	7100 5300 6800 5300
+Wire Wire Line
+	6800 5225 6800 5300
 $EndSCHEMATC
