File: fwr/fwr.2sch.sch (KiCad schematic (older format))
At the start: 36 parts, among them J1 CV_Input, J2 Input, J3 Synth_power_2x5, J4 Output, U1 TL074

Commit message: xor
Parts:
- Bias1, CV_Amount1, Feedback1: symbol Device:R_Potentiometer -> fwr.2sch-rescue:R_Potentiometer-Device
- C5, C6: symbol Device:C_Polarized -> fwr.2sch-rescue:C_Polarized-Device
- FB1, FB2: symbol Device:FerriteBead -> fwr.2sch-rescue:FerriteBead-Device
- J1, J2, J4: symbol 2_pin_molex_connector:2_pin_Molex_connector -> fwr.2sch-rescue:2_pin_Molex_connector-2_pin_molex_connector
- J3: symbol synth_power_2x5:Synth_power_2x5 -> fwr.2sch-rescue:Synth_power_2x5-synth_power_2x5
Changed lines of the file:
@@
 $EndComp
 $Comp
-L 2_pin_molex_connector:2_pin_Molex_connector J2
+L fwr.2sch-rescue:2_pin_Molex_connector-2_pin_molex_connector J2
 U 1 1 60E3FD0B
 P 2650 2225
@@
 $EndComp
 $Comp
-L 2_pin_molex_connector:2_pin_Molex_connector J1
+L fwr.2sch-rescue:2_pin_Molex_connector-2_pin_molex_connector J1
 U 1 1 60E42009
 P 2150 3700
@@
 $EndComp
 $Comp
-L 2_pin_molex_connector:2_pin_Molex_connector J4
+L fwr.2sch-rescue:2_pin_Molex_connector-2_pin_molex_connector J4
 U 1 1 60E4264B
 P 8975 3575
@@
 Connection ~ 6700 3300
 $Comp
-L Device:R_Potentiometer Bias1
+L fwr.2sch-rescue:R_Potentiometer-Device Bias1
 U 1 1 60E94F16
 P 2675 2900
@@
 $EndComp
 $Comp
-L Device:R_Potentiometer CV_Amount1
+L fwr.2sch-rescue:R_Potentiometer-Device CV_Amount1
 U 1 1 60EA23B3
 P 2900 4075
@@
 	2900 3700 2350 3700
 $Comp
-L Device:R_Potentiometer Feedback1
+L fwr.2sch-rescue:R_Potentiometer-Device Feedback1
 U 1 1 60EB2357
 P 2400 1600
@@
 Connection ~ 8550 3575
 $Comp
-L synth_power_2x5:Synth_power_2x5 J3
+L fwr.2sch-rescue:Synth_power_2x5-synth_power_2x5 J3
 U 1 1 60ECEDE7
 P 5425 5450
@@
 $EndComp
 $Comp
-L Device:FerriteBead FB2
+L fwr.2sch-rescue:FerriteBead-Device FB2
 U 1 1 60EF236A
 P 6300 5125
@@
 $EndComp
 $Comp
-L Device:FerriteBead FB1
+L fwr.2sch-rescue:FerriteBead-Device FB1
 U 1 1 60EF8676
 P 6275 6000
@@
 	5875 6000 6125 6000
 $Comp
-L Device:C_Polarized C6
+L fwr.2sch-rescue:C_Polarized-Device C6
 U 1 1 60F04170
 P 6650 5850
@@
 $EndComp
 $Comp
-L Device:C_Polarized C5
+L fwr.2sch-rescue:C_Polarized-Device C5
 U 1 1 60F05829
 P 6650 5175
