File: wahwah/wahwah/wahwah.kicad_pcb (KiCad board)
At the start: 2 copper layers, 50 x 200 mm, 57 parts, among them J1 Input, J2 Synth_power_2x5, J3 Output, J4 CV_switched_jack, Q1 S8050, Q2 S8050, SW1 SW_DPDT_x2, U1 TL074, U5 VTL5C, U6 VTL5C

Commit message: eyeyey
Parts:
- removed Cutoff1, LfoRate1: 100K, ao_tht:Potentiometer_Alpha_RD901F-40-00D_Single_Vertical_CircularHoles_centered
- removed L1: 200mH, digikey-footprints:Inductor_13R106C
- removed the R21 at (62.1, 55.1)
- removed the R24 at (29.9, 80.9)
- removed R7: 150K, ao_tht:R_Axial_DIN0207_L6.3mm_D2.5mm_P7.62mm_Horizontal
- removed U5, U6: VTL5C, OptoDevice:PerkinElmer_VTL5C
- added Attenuate: 100K, ao_tht:Potentiometer_Alpha_RD901F-40-00D_Single_Vertical_CircularHoles_centered, B.Cu at (-526.5, 88.0)
- added Cutoff: 100K, ao_tht:Potentiometer_Alpha_RD901F-40-00D_Single_Vertical_CircularHoles_centered, B.Cu at (-550.0, -1.00)
- added D4: LED, ao_tht:LED_D5.0mm, B.Cu at (-548.5, 68.0)
- added G***: LOGO, ao_tht:wahwah, B.Cu at (-550.0, 19.5)
- added G***: LOGO, ao_tht:goose, B.Cu at (-551.5, -19.0)
- added G***: LOGO, ao_tht:keystone, F.Cu at (-542.0, -18.0)
- added Inductor: 200mH or 500mH (We like 200, use sockets), digikey-footprints:Inductor_13R106C, F.Cu at (-524.0, 68.5)
- added LFO Rate: 100K, ao_tht:Potentiometer_Alpha_RD901F-40-00D_Single_Vertical_CircularHoles_centered, B.Cu at (-573.5, 88.0)
- added Q: 100K, ao_tht:Potentiometer_Alpha_RD901F-40-00D_Single_Vertical_CircularHoles_centered, B.Cu at (-526.5, 48.0)
- added R21: 150K, ao_tht:R_Axial_DIN0207_L6.3mm_D2.5mm_P7.62mm_Horizontal, F.Cu at (-536.5, 50.5)
- added R21: 47K, ao_tht:R_Axial_DIN0207_L6.3mm_D2.5mm_P7.62mm_Horizontal, F.Cu at (-584.5, 54.0)
- added R24: 10K, ao_tht:R_Axial_DIN0207_L6.3mm_D2.5mm_P7.62mm_Horizontal, F.Cu at (-584.0, 25.5)
- added R24: 1K, ao_tht:R_Axial_DIN0207_L6.3mm_D2.5mm_P7.62mm_Horizontal, F.Cu at (-541.0, 65.5)
- added TP1: TestPoint, ao_tht:Perf_Board_Hole, F.Cu at (-566.5, 62.0)
- added TP2: TestPoint, ao_tht:Perf_Board_Hole, F.Cu at (-580.5, 62.0)
- added TrimNeg: 20K, ao_tht:Potentiometer_Bourns_3296W_Vertical, F.Cu at (-550.0, 24.5)
- added TrimPos: 20K, ao_tht:Potentiometer_Bourns_3296W_Vertical, F.Cu at (-550.0, 13.5)
- added VTL5C or DIY: VTL5C, OptoDevice:PerkinElmer_VTL5C, F.Cu at (-572.0, 62.0)
- added VTL5C or DIY: VTL5C, OptoDevice:PerkinElmer_VTL5C, F.Cu at (-558.0, 62.0)
- C1, C10, C5, C6, C8, C9: footprint ao_tht:C_Disc_D3.0mm_W1.6mm_P2.50mm -> ao_tht:C_Rect_L7.2mm_W2.5mm_P5.00mm_FKS2_FKP2_MKS2_MKP2
- C2: value .01uf -> .033uf USE SOCKETS!; footprint ao_tht:C_Disc_D3.0mm_W1.6mm_P2.50mm -> ao_tht:C_Rect_L7.2mm_W2.5mm_P5.00mm_FKS2_FKP2_MKS2_MKP2
- C7: value .033uf -> .01uf; footprint ao_tht:C_Disc_D3.0mm_W1.6mm_P2.50mm -> ao_tht:C_Rect_L7.2mm_W2.5mm_P5.00mm_FKS2_FKP2_MKS2_MKP2
- J1, J3, J4: moved to F.Cu
- moved H2 683.9 mm to (-593.5, -24.0)
- moved C7 677.9 mm to (-591.0, 48.5)
- moved C5 677.7 mm to (-591.0, 60.0)
- moved Q1 674.1 mm to (-590.5, 8.50), turned to 90 degrees
- moved C2 670.5 mm to (-583.0, 35.5)
- moved Q2 664.5 mm to (-590.5, 32.5), turned to 90 degrees
- moved R1 653.3 mm to (-576.5, -20.5), turned to 180 degrees
- moved R23 646.8 mm to (-584.5, 70.2), turned to 180 degrees
- moved C6 645.8 mm to (-577.5, -0.50), turned to 180 degrees
- moved R16 642.4 mm to (-592.5, 43.0)
- moved R15 639.3 mm to (-560.0, 86.0), turned to 270 degrees
- moved R28 638.4 mm to (-576.5, -15.5), turned to 180 degrees
- moved R19 633.2 mm to (-584.0, 10.5)
- moved R22 630.0 mm to (-584.0, -4.50)
- moved R17 629.3 mm to (-584.0, 5.50)
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Connections:
- D3 pad 1: X -> Net-(ATTN1-Pad2)
- J4 pad 1: GND -> Net-(D3-Pad2)
- J4 pad 2: Net-(D3-Pad2) -> Net-(C1-Pad1)
- J4 pad 3: Net-(C1-Pad1) -> GND
- Q1 pad 2: Net-(C2-Pad1) -> Net-(C7-Pad1)
- Q2 pad 1: Net-(C7-Pad1) -> Net-(C2-Pad1)
- R16 pad 1: Net-(C2-Pad2) -> Net-(C7-Pad2)
- R17 pad 1: Net-(C2-Pad1) -> Net-(C7-Pad1)
- R17 pad 2: Net-(C7-Pad2) -> Net-(C2-Pad2)
- R26 pad 2: B -> A
- R27 pad 2: A -> B
- R29 pad 1: Net-(C7-Pad1) -> Net-(C2-Pad1)
Routing:
- net Net-(R1-Pad1): track 0.00 -> 138.8 mm
- net Net-(C1-Pad2): track 0.00 -> 127.9 mm
- net Net-(J1-Pad1): track 0.00 -> 117.8 mm
- net Net-(C2-Pad2): track 0.00 -> 113.8 mm
- net I: track 0.00 -> 104.9 mm
- net X: track 0.00 -> 94.6 mm
- net Net-(R11-Pad1): track 0.00 -> 90.7 mm
- net Net-(C4-Pad2): track 0.00 -> 88.2 mm
- net Net-(C5-Pad2): track 0.00 -> 87.6 mm
- net Net-(C6-Pad2): track 0.00 -> 86.9 mm
- net Net-(C1-Pad1): track 0.00 -> 79.7 mm
- net Net-(R3-Pad1): track 0.00 -> 76.6 mm
- net B: track 0.00 -> 72.9 mm
- net Net-(LfoRate1-Pad3): track 0.00 -> 69.4 mm
- net Net-(R5-Pad1): track 0.00 -> 63.0 mm
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- added copper zone on B.Cu, net +12V
- added copper zone on F.Cu, net GND
Other:
- board size 50 x 200 mm -> 98 x 130 mm
- board text added: "Callibrate LFO with TP1/2"
- board text added: "LDR side"
- board text added: "LED side"
- board text added: "Use with distortion for maximum fun!"
- board text added: "WW847 PCB v0.1"
- board text added: "Wah Wah!"
- board text added: "based on the Vox V847"
- board text added: "by Rich and Martin Jones designed in Pennsylvania, 2021"
