File: wahwah/wahwah/wahwah.sch (KiCad schematic (older format))
At the start: 57 parts, among them J1 Input, J2 Synth_power_2x5, J3 Output, J4 CV_switched_jack, Q1 S8050, Q2 S8050, SW1 SW_DPDT_x2, U1 TL074, U5 VTL5C, U6 VTL5C

Commit message: eyeyey
Parts:
- removed R21: 47K, ao_tht:R_Axial_DIN0207_L6.3mm_D2.5mm_P7.62mm_Horizontal, symbol Device:R
- removed R25: 10K, ao_tht:R_Axial_DIN0207_L6.3mm_D2.5mm_P7.62mm_Horizontal, symbol Device:R
- added ATTN1, Q3: 100K, ao_tht:Potentiometer_Alpha_RD901F-40-00D_Single_Vertical_CircularHoles_centered, symbol Device:R_Potentiometer
- added D4: LED, ao_tht:LED_D5.0mm, symbol Device:LED
- added TP1, TP2: TestPoint, ao_tht:Perf_Board_Hole, symbol Connector:TestPoint
- added TrimNeg1, Trimpos1: 20K, ao_tht:Potentiometer_Bourns_3296W_Vertical, symbol Device:R_Potentiometer
- C1, C10, C5, C6, C8, C9: footprint ao_tht:C_Disc_D3.0mm_W1.6mm_P2.50mm -> ao_tht:C_Rect_L7.2mm_W2.5mm_P5.00mm_FKS2_FKP2_MKS2_MKP2
- C2: renamed from C7; value .033uf -> .033uf USE SOCKETS!; footprint ao_tht:C_Disc_D3.0mm_W1.6mm_P2.50mm -> ao_tht:C_Rect_L7.2mm_W2.5mm_P5.00mm_FKS2_FKP2_MKS2_MKP2
- C7: renamed from C2; footprint ao_tht:C_Disc_D3.0mm_W1.6mm_P2.50mm -> ao_tht:C_Rect_L7.2mm_W2.5mm_P5.00mm_FKS2_FKP2_MKS2_MKP2
- R24: value 10K -> 1K
- renumbered R7 to R21
Connections:
- net +12V: now also Trimpos1.1, Trimpos1.2; no longer R24.2
- net A: now also R26.2, Trimpos1.3; no longer R27.2
- net B: now also R27.2, TrimNeg1.3; no longer R24.1, R26.2
- net GND: now also J4.3 (Pin_3), R24.2, ATTN1.3; no longer J4.1 (Pin_1)
- net X: now also ATTN1.1, D4.2 (A); no longer D3.1 (K)
- net at C4.2, C9.2, D1.2 (A)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: now also TrimNeg1.1, TrimNeg1.2
- net at R11.1, U1.1, U5.1 (-): now also TP2.1
- net at R12.1, U1.7, U6.2 (+): now also TP1.1
- net at C1.1, R9.1, U1.14: now also J4.2 (Pin_2); no longer J4.3 (Pin_3)
- net at C2.2, L1.2, R17.2: now also Q3.1, Q3.2
- net at C5.2, L1.1, R20.2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: now also Q3.3
- net at D3.2 (A): now also J4.1 (Pin_1); no longer J4.2 (Pin_2)
- new net: D4.1 (K), R24.1
- new net: ATTN1.2, D3.1 (K)
Other:
- note added: "LFO / CV In"
- note added: "TODO: Is vactrol backwrds"
- note removed: "LFO"
- moved on the sheet: J4
