File: sub/sub_destroyer/sub_destroyer.sch (KiCad schematic (older format))
At the start: 32 parts

Commit message: sub work
Parts:
- removed R?: 220K, symbol Device:R
- removed R? (x4): 330R, symbol Device:R
- removed U?: TL074, symbol 4xxx:4013
- added -1RMP, -1SQR, -2PULSE, -2SQR: A100K, symbol Device:R_POT
- added CP?: 470nf, symbol Device:CP1
- added D?: LED, symbol Device:LED
- added J?: Synth_power_2x5, ao_tht:Power_Header, symbol ao_tht:Synth_power_2x5
- added J?: OUTPUT, symbol sub_destroyer-rescue:2_pin_Molex_connector-2_pin_molex_connector
- added R15: 100K, ao_tht:R_Axial_DIN0207_L6.3mm_D2.5mm_P10.16mm_Horizontal, symbol ao_tht:R
- added R16, R18: 100K, symbol Device:R
- added R17: 51K, symbol Device:R
- added R?: 10K, ao_tht:R_Axial_DIN0207_L6.3mm_D2.5mm_P10.16mm_Horizontal, symbol ao_tht:R
- added R?: 330R, symbol Device:R
- added R?: 1K, symbol Device:R
- added RAMPTRIM1: 100K, symbol Device:R_POT_TRIM
- added RV?: MASTER, symbol Device:R_POT
- added U? (x3): TL072, symbol Amplifier_Operational:TL072
- added U?: LM4040LP-5, ao_tht:TO-92_Inline_Wide, symbol ao_tht:LM4040LP-5
- added U?: CD4013, symbol 4xxx:4013
- J1: renamed from J?; symbol 2_pin_molex_connector:2_pin_Molex_connector -> sub_destroyer-rescue:2_pin_Molex_connector-2_pin_molex_connector
- R11, R7, R9: renamed from R?; value 300K -> 100K
- R14: renamed from R?; value 150K -> 50K
- gave numbers to parts that had none: 16
Connections:
- net GND: now also U2.10 (+), U2.12 (+), U2.3 (+), U2.5 (+), -1RMP.1, -1SQR.1, -2PULSE.1, -2SQR.1, CP?.2, D?.1 (K), J?.2 (Pin_2), U?.2 (K), U?.3 (+); no longer R3.2
- net at J1.1 (Pin_1), R1.2: now also R13.2
- net at R4.2, U1.13 (Q), U1.3 (C): now also RAMPTRIM1.1, RAMPTRIM1.2
- net at U2.1: now also -1SQR.3, R15.1
- net at R7.1, U2.2 (-): now also R6.1, R15.2
- net at R9.1, U2.6 (-): now also R8.1, R18.2
- net at U2.7: now also -2PULSE.3, R18.1
- net at U2.8: now also -2SQR.3, R16.1
- net at R11.1, U2.9 (-): now also R10.1, R16.2
- net at R14.1, U2.13 (-): now also R12.1, R13.1, R17.2
- net at U2.14: now also -1RMP.3, R17.1
- net VNEGFIVE: now reaches R7.2
- net VNEGFIVE: now also R11.2, R14.2, R9.2, CP?.1, R?.2, U?.3 (A)
- net at R12.2: now also RAMPTRIM1.3
- new net: -1RMP.2, -1SQR.2, -2PULSE.2, -2SQR.2, RV?.1, U?.2 (-), U?.5 (+)
- new net: R?.1, RV?.2, RV?.3, U?.1
- new net: R?.1, U?.6 (-), U?.7
- new net: D?.2 (A), R?.2
- new net: J?.1 (Pin_1), R?.2
- new net V+12: R3.2
- new net VNEGTWELVE: R?.1
Other:
- note added: "via https://bgr360.github.io/assets/pdf/mutable_instruments/grids_v02.pdf"
- note removed: "TODO: Diode protection for 2n3904"
- moved on the sheet: D1, D2, D3, J1, Q1, R1, R10, R11, R12, R13, R14, R2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

Commit message: sub
Parts:
- added C1, C2: 10uf, ao_tht:CP_Radial_D5.0mm_P2.00mm, symbol Device:CP
- added C3, C4, C5, C6, C7: 100nf, ao_tht:C_Disc_D3.0mm_W1.6mm_P2.50mm, symbol ao_tht:C
- added D4, D5: 1N4148, Diode_THT:D_DO-35_SOD27_P7.62mm_Horizontal, symbol Device:D
- added D7: PWR_LED, ao_tht:LED_D5.0mm, symbol Device:LED
- added R22: 1K, ao_tht:R_Axial_DIN0207_L6.3mm_D2.5mm_P7.62mm_Horizontal, symbol ao_tht:R
- added R23, R24, R25, R26: 10K, ao_tht:R_Axial_DIN0207_L6.3mm_D2.5mm_P7.62mm_Horizontal, symbol ao_tht:R
- added SW1: ONOFF_SW, ao_tht:DPDT-toggle-switch-1M-seriesx, symbol Switch:SW_DPDT_x2
- CP1: renamed from CP?; footprint (none) -> ao_tht:CP_Radial_D5.0mm_P2.00mm
- D6: renamed from D?; value LED -> SIG_LED; footprint (none) -> ao_tht:LED_D5.0mm
- J1: footprint (none) -> ao_tht:Molex_KK-254_AE-6410-02A_1x02_P2.54mm_Vertical
- J3: renamed from J?; footprint (none) -> ao_tht:Molex_KK-254_AE-6410-02A_1x02_P2.54mm_Vertical
- R1, R10, R11, R12, R13, R16, R17, R18, R2, R3, R4, R5, R6, R7, R8, R9: footprint (none) -> ao_tht:R_Axial_DIN0207_L6.3mm_D2.5mm_P7.62mm_Horizontal
- R14: value 50K -> 51K; footprint (none) -> ao_tht:R_Axial_DIN0207_L6.3mm_D2.5mm_P7.62mm_Horizontal
- R15: footprint ao_tht:R_Axial_DIN0207_L6.3mm_D2.5mm_P10.16mm_Horizontal -> ao_tht:R_Axial_DIN0207_L6.3mm_D2.5mm_P7.62mm_Horizontal
- R19: renamed from R?; footprint ao_tht:R_Axial_DIN0207_L6.3mm_D2.5mm_P10.16mm_Horizontal -> ao_tht:R_Axial_DIN0207_L6.3mm_D2.5mm_P7.62mm_Horizontal
- R20: renamed from R?; footprint (none) -> ao_tht:R_Axial_DIN0207_L6.3mm_D2.5mm_P7.62mm_Horizontal
- R21: renamed from R?; value 330R -> 1K; footprint (none) -> ao_tht:R_Axial_DIN0207_L6.3mm_D2.5mm_P7.62mm_Horizontal
- RAMPTRIM1: footprint (none) -> ao_tht:Potentiometer_Bourns_3296W_Vertical
- RV1: renamed from -1RMP; value A100K -> -1RMP 100K; footprint (none) -> ao_tht:Potentiometer_Alpha_RD901F-40-00D_Single_Vertical_CircularHoles_centered
- RV2: renamed from -2SQR; value A100K -> -2SQR 100K; footprint (none) -> ao_tht:Potentiometer_Alpha_RD901F-40-00D_Single_Vertical_CircularHoles_centered
- RV3: renamed from -2PULSE; value A100K -> -2PLS 100K; footprint (none) -> ao_tht:Potentiometer_Alpha_RD901F-40-00D_Single_Vertical_CircularHoles_centered
- RV4: renamed from -1SQR; value A100K -> -1SQR 100K; footprint (none) -> ao_tht:Potentiometer_Alpha_RD901F-40-00D_Single_Vertical_CircularHoles_centered
- RV5: renamed from RV?; value MASTER -> 10K; footprint (none) -> ao_tht:Potentiometer_Alpha_RD901F-40-00D_Single_Vertical_CircularHoles
- U1, U2: footprint (none) -> ao_tht:DIP-14_W7.62mm_Socket_LongPads
- U1: renamed from U?; footprint (none) -> ao_tht:DIP-14_W7.62mm_Socket_LongPads
- U4: renamed from U?; footprint (none) -> ao_tht:DIP-8_W7.62mm_Socket_LongPads
- gave numbers to parts that had none: 2
Connections:
- net V+12 is gone; now on an unnamed net: R3.2
- net VNEGTWELVE is gone; now on an unnamed net: R19.1
- net GND: now also J2.3 (GND), J2.4 (GND), J2.5 (GND), J2.6 (GND), J2.7 (GND), J2.8 (GND), R21.2, U1.7 (VSS), C1.2, C2.1, C3.1, C4.2, C5.1, C6.2, C7.1, R22.1; no longer D6.1 (K)
- net at J1.1 (Pin_1), R1.2, R13.2: now also SW1.6 (C)
- net at U1.2 (~Q): now also U1.5 (D)
- net at U2.11 (V-): now also U4.4 (V-), C2.2, C4.1, C6.1, D5.2 (A)
- net at U2.4 (V+): now also U1.14 (VDD), U4.8 (V+), C1.1, C3.2, C5.2, C7.2, D4.1 (K), SW1.2 (B)
- net at R21.1, U4.7: now also D6.2 (A); no longer U4.6 (-)
- net at J2.1 (-12V): now also J2.2 (-12V), D5.1 (K)
- net at J2.10 (+12V): now also J2.9 (+12V), D4.2 (A)
- net at R20.2: now also U4.5 (+), SW1.4 (A); no longer J3.1 (Pin_1)
- net VNEGFIVE: no longer names the net of CP1.1, R11.2, R14.2, R19.2, R7.2, R9.2, U3.3 (A)
- new net: R23.2, RV4.2
- new net: R24.2, RV3.2
- new net: R25.2, RV2.2
- new net: R26.2, RV1.2
- new net: R23.1, R24.1, R25.1, R26.1, RV5.1, U4.2 (-)
- new net: D6.1 (K), U4.6 (-)
- new net: J3.1 (Pin_1), SW1.5 (B)
- new net: D7.2 (A), SW1.1 (A)
- new net: D7.1 (K), R22.2
- no-connect marks 0 -> 1
Other:
- note added: "\n"
- moved on the sheet: D6, J2, J3, U1C, U2E, U4C

Commit message: routed
Parts:
- C3, C4, C5, C6, C7: footprint ao_tht:C_Disc_D3.0mm_W1.6mm_P2.50mm -> ao_tht:C_Rect_L7.2mm_W2.5mm_P5.00mm_FKS2_FKP2_MKS2_MKP2
Connections:
- net at D6.1 (K), U4.6 (-): now also R21.1
- net at D6.2 (A), U4.7: no longer R21.1
Other:
- note added: "TODO confirm this"
- note added: "TODO confirm this?"
- moved on the sheet: D6, R21
Changed lines of the file:
@@
 L Device:LED D6
 U 1 1 61E4F139
-P 9900 2975
-F 0 "D6" H 9893 2720 50  0000 C CNN
-F 1 "SIG_LED" H 9893 2811 50  0000 C CNN
-F 2 "ao_tht:LED_D5.0mm" H 9900 2975 50  0001 C CNN
-F 3 "~" H 9900 2975 50  0001 C CNN
-	1    9900 2975
-	1    0    0    -1
+P 10375 3425
+F 0 "D6" H 10368 3170 50  0000 C CNN
+F 1 "SIG_LED" H 10368 3261 50  0000 C CNN
+F 2 "ao_tht:LED_D5.0mm" H 10375 3425 50  0001 C CNN
+F 3 "~" H 10375 3425 50  0001 C CNN
+	1    10375 3425
+	-1   0    0    1
 $EndComp
 $Comp
 L Device:R R21
 U 1 1 61E51035
-P 10500 3425
-F 0 "R21" V 10707 3425 50  0000 C CNN
-F 1 "1K" V 10616 3425 50  0000 C CNN
-F 2 "ao_tht:R_Axial_DIN0207_L6.3mm_D2.5mm_P7.62mm_Horizontal" V 10430 3425 50  0001 C CNN
-F 3 "~" H 10500 3425 50  0001 C CNN
-	1    10500 3425
+P 10825 3425
+F 0 "R21" V 11032 3425 50  0000 C CNN
+F 1 "1K" V 10941 3425 50  0000 C CNN
+F 2 "ao_tht:R_Axial_DIN0207_L6.3mm_D2.5mm_P7.62mm_Horizontal" V 10755 3425 50  0001 C CNN
+F 3 "~" H 10825 3425 50  0001 C CNN
+	1    10825 3425
 	0    -1   -1   0
 $EndComp
@@
 L power:GND #PWR030
 U 1 1 61E521B0
-P 10700 3425
-F 0 "#PWR030" H 10700 3175 50  0001 C CNN
-F 1 "GND" H 10705 3252 50  0000 C CNN
-F 2 "" H 10700 3425 50  0001 C CNN
-F 3 "" H 10700 3425 50  0001 C CNN
-	1    10700 3425
-	1    0    0    -1
-$EndComp
-Wire Wire Line
-	10650 3425 10700 3425
+P 11025 3425
+F 0 "#PWR030" H 11025 3175 50  0001 C CNN
+F 1 "GND" H 11030 3252 50  0000 C CNN
+F 2 "" H 11025 3425 50  0001 C CNN
+F 3 "" H 11025 3425 50  0001 C CNN
+	1    11025 3425
+	1    0    0    -1
+$EndComp
+Wire Wire Line
+	10975 3425 11025 3425
 $Comp
 L sub_destroyer-rescue:2_pin_Molex_connector-2_pin_molex_connector J3
@@
 F 0 "C3" H 3090 6196 50  0000 L CNN
 F 1 "100nf" H 3090 6105 50  0000 L CNN
-F 2 "ao_tht:C_Disc_D3.0mm_W1.6mm_P2.50mm" H 3013 6000 50  0001 C CNN
+F 2 "ao_tht:C_Rect_L7.2mm_W2.5mm_P5.00mm_FKS2_FKP2_MKS2_MKP2" H 3013 6000 50  0001 C CNN
 F 3 "" H 2975 6150 50  0001 C CNN
 F 4 "Tayda" H 2975 6150 50  0001 C CNN "Vendor"
@@
 F 0 "C7" H 4065 6196 50  0000 L CNN
 F 1 "100nf" H 4065 6105 50  0000 L CNN
-F 2 "ao_tht:C_Disc_D3.0mm_W1.6mm_P2.50mm" H 3988 6000 50  0001 C CNN
+F 2 "ao_tht:C_Rect_L7.2mm_W2.5mm_P5.00mm_FKS2_FKP2_MKS2_MKP2" H 3988 6000 50  0001 C CNN
 F 3 "" H 3950 6150 50  0001 C CNN
 F 4 "Tayda" H 3950 6150 50  0001 C CNN "Vendor"
@@
 F 0 "C5" H 3565 6196 50  0000 L CNN
 F 1 "100nf" H 3565 6105 50  0000 L CNN
-F 2 "ao_tht:C_Disc_D3.0mm_W1.6mm_P2.50mm" H 3488 6000 50  0001 C CNN
+F 2 "ao_tht:C_Rect_L7.2mm_W2.5mm_P5.00mm_FKS2_FKP2_MKS2_MKP2" H 3488 6000 50  0001 C CNN
 F 3 "" H 3450 6150 50  0001 C CNN
 F 4 "Tayda" H 3450 6150 50  0001 C CNN "Vendor"
@@
 F 0 "C4" H 3090 7396 50  0000 L CNN
 F 1 "100nf" H 3090 7305 50  0000 L CNN
-F 2 "ao_tht:C_Disc_D3.0mm_W1.6mm_P2.50mm" H 3013 7200 50  0001 C CNN
+F 2 "ao_tht:C_Rect_L7.2mm_W2.5mm_P5.00mm_FKS2_FKP2_MKS2_MKP2" H 3013 7200 50  0001 C CNN
 F 3 "" H 2975 7350 50  0001 C CNN
 F 4 "Tayda" H 2975 7350 50  0001 C CNN "Vendor"
@@
 F 0 "C6" H 3565 7396 50  0000 L CNN
 F 1 "100nf" H 3565 7305 50  0000 L CNN
-F 2 "ao_tht:C_Disc_D3.0mm_W1.6mm_P2.50mm" H 3488 7200 50  0001 C CNN
+F 2 "ao_tht:C_Rect_L7.2mm_W2.5mm_P5.00mm_FKS2_FKP2_MKS2_MKP2" H 3488 7200 50  0001 C CNN
 F 3 "" H 3450 7350 50  0001 C CNN
 F 4 "Tayda" H 3450 7350 50  0001 C CNN "Vendor"
@@
 NoConn ~ 4700 5875
 Wire Wire Line
-	10150 3425 10250 3425
-Wire Wire Line
-	10250 3425 10250 2975
-Wire Wire Line
-	10250 2975 10050 2975
-Connection ~ 10250 3425
-Wire Wire Line
-	10250 3425 10350 3425
-Wire Wire Line
-	9750 2975 9550 2975
-Wire Wire Line
-	9550 2975 9550 3325
-Wire Wire Line
 	8575 2375 9150 2375
 Wire Wire Line
@@
 Wire Wire Line
 	7975 4250 7700 4250
+Text Notes 2275 4550 0    50   ~ 0
+TODO confirm this
+Text Notes 4600 7150 0    50   ~ 0
+TODO confirm this?
+Wire Wire Line
+	10150 3425 10225 3425
+Wire Wire Line
+	10525 3425 10600 3425
+Wire Wire Line
+	10600 3425 10600 3025
+Wire Wire Line
+	10600 3025 9525 3025
+Wire Wire Line
+	9525 3025 9525 3325
+Wire Wire Line
+	9525 3325 9550 3325
+Connection ~ 10600 3425
+Wire Wire Line
+	10600 3425 10675 3425
 $EndSCHEMATC
