File: sub/sub_destroyer/sub_destroyer.kicad_pcb (KiCad board)
At the start: 2 copper layers, 49 x 150.5 mm, 58 parts, among them J1 INPUT, J2 Synth_power_2x5, J3 OUTPUT, Q1 2N3904, SW1 ONOFF_SW, U1 CD4013, U2 TL074, U3 LM4040LP-5, U4 TL072

Commit message: routed
Parts:
- C3, C4, C5, C6, C7: footprint ao_tht:C_Disc_D3.0mm_W1.6mm_P2.50mm -> ao_tht:C_Rect_L7.2mm_W2.5mm_P5.00mm_FKS2_FKP2_MKS2_MKP2
- moved R13 150.5 mm to (193.5, 133.0)
- moved R1 124.4 mm to (193.5, 126.5)
- moved R17 123.9 mm to (159.5, 42.0)
- moved R7 123.4 mm to (159.5, 47.5)
- moved R15 123.0 mm to (159.5, 53.0)
- moved R12 122.8 mm to (159.5, 31.0)
- moved R6 122.6 mm to (159.5, 58.5)
- moved R14 122.4 mm to (159.5, 36.5)
- moved R9 122.2 mm to (159.5, 63.5)
- moved R8 104.9 mm to (193.5, 85.0)
- moved D3 104.4 mm to (193.5, 90.5)
- moved D2 104.1 mm to (193.5, 95.5)
- moved R4 103.6 mm to (193.5, 101.0)
- moved R10 103.4 mm to (193.5, 106.5)
- moved R5 102.7 mm to (193.5, 112.5)
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Connections:
- R21 pad 1: Net-(D6-Pad2) -> Net-(D6-Pad1)
Routing:
- net Net-(R24-Pad2): track 0.00 -> 398.0 mm
- net GND: track 0.00 -> 237.3 mm, vias 0 -> 4
- net Net-(C2-Pad2): track 0.00 -> 162.2 mm, vias 0 -> 4
- net Net-(R23-Pad1): track 0.00 -> 135.7 mm, vias 0 -> 5
- net Net-(R12-Pad1): track 0.00 -> 124.9 mm, vias 0 -> 1
- net Net-(CP1-Pad1): track 0.00 -> 122.2 mm
- net Net-(Q1-Pad3): track 0.00 -> 113.5 mm
- net Net-(R4-Pad2): track 0.00 -> 97.7 mm
- net Net-(D2-Pad2): track 0.00 -> 96.2 mm, vias 0 -> 2
- net Net-(R15-Pad1): track 0.00 -> 95.9 mm
- net Net-(C1-Pad1): track 0.00 -> 90.4 mm, vias 0 -> 2
- net Net-(R18-Pad2): track 0.00 -> 79.5 mm, vias 0 -> 4
- net Net-(D1-Pad1): track 0.00 -> 79.1 mm
- net Net-(R10-Pad1): track 0.00 -> 77.3 mm
- net Net-(R18-Pad1): track 0.00 -> 72.7 mm
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
Commit message: nice
Routing:
- net Net-(R24-Pad2): track 398.0 -> 76.9 mm
Other:
- board text added: "Sub Destroyer v0.1 Rich Jones @BlackDeath help from @AnalogOutput & @Sonosus based on ElectricDruid Dec 2021"

Commit message: envy
Parts:
- added G***: LOGO, ao_tht:BD3, B.Cu at (197.7, 91.1)
- added G***: LOGO, ao_tht:sd5, B.Cu at (163.3, 70.8)
- renumbered J1 to Input, J3 to Output
Other:
- board text added: "Designed in Bergen, Norway"

Commit message: blah
Parts:
- removed REF** (x2): Kosmo_Jack_Hole, ao_panel:Kosmo_Jack_Hole
Other:
- board text added: "JLCJLCJLCJLC"
