File: sub/sub_destroyer/sub_destroyer_panel.kicad_pcb (KiCad board)
At the start: 2 copper layers, 50 x 200 mm, 30 parts

Commit message: envy
Parts:
- removed the G*** at (213.5, 92.4)
- added G***: LOGO, ao_tht:2pl3, B.Cu at (215.0, 126.3)
- moved G*** 34.0 mm to (214.2, 92.5)
Routing:
- added copper zone on B.Cu, net (none)
- added copper zone on F.Cu, net (none)
Other:
- board text added: "JLCJLCJLCJLC"
Changed lines of the file:
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@@
   (general
     (thickness 1.6)
-    (drawings 4)
+    (drawings 5)
     (tracks 0)
     (zones 0)
@@
   (page A4)
   (layers
-    (0 F.Cu signal)
-    (31 B.Cu signal)
+    (0 F.Cu signal hide)
+    (31 B.Cu signal hide)
     (32 B.Adhes user)
     (33 F.Adhes user)
@@
     (uvia_dia 0.3)
     (uvia_drill 0.1)
+  )
+  (module ao_tht:2pl3 (layer B.Cu)
+    (at 215 126.3 180)
+    (fp_text reference G*** (at 0 0) (layer B.SilkS) hide
+      (effects (font (size 1.524 1.524) (thickness 0.3)) (justify mirror))
+    )
+    (fp_text value LOGO (at 0.75 0) (layer B.SilkS) hide
+      (effects (font (size 1.524 1.524) (thickness 0.3)) (justify mirror))
+    )
+    (fp_poly (pts (xy -3.299577 2.234498) (xy -2.765598 1.896093) (xy -2.423912 1.414765) (xy -2.343321 0.823113)
+      (xy -2.375307 0.648466) (xy -2.565471 0.213696) (xy -2.884152 -0.265784) (xy -2.930717 -0.32279)
+      (xy -3.215465 -0.686378) (xy -3.367157 -0.929149) (xy -3.374825 -0.958158) (xy -3.218495 -1.029299)
+      (xy -2.834153 -1.064818) (xy -2.753146 -1.065734) (xy -2.335465 -1.095439) (xy -2.164149 -1.246111)
+      (xy -2.131468 -1.598601) (xy -2.131468 -2.131468) (xy -3.907692 -2.131468) (xy -4.653289 -2.118451)
+      (xy -5.244773 -2.083352) (xy -5.60696 -2.0321) (xy -5.683916 -1.991392) (xy -5.573219 -1.804709)
+      (xy -5.276908 -1.42297) (xy -4.848651 -0.913685) (xy -4.618181 -0.650734) (xy -4.144202 -0.090624)
+      (xy -3.778591 0.391217) (xy -3.575934 0.720534) (xy -3.552447 0.798965) (xy -3.701379 1.118254)
+      (xy -4.080846 1.272686) (xy -4.589853 1.225027) (xy -4.652837 1.20466) (xy -5.134187 1.144946)
+      (xy -5.492777 1.281589) (xy -5.668196 1.54174) (xy -5.600031 1.85255) (xy -5.367246 2.066156)
+      (xy -4.669204 2.352131) (xy -3.957046 2.397377) (xy -3.299577 2.234498)) (layer B.SilkS) (width 0.01))
+    (fp_poly (pts (xy 0.490569 2.271668) (xy 1.097537 2.211013) (xy 1.427639 2.12871) (xy 1.96605 1.753112)
+      (xy 2.244111 1.235577) (xy 2.283467 0.650218) (xy 2.105766 0.071149) (xy 1.732651 -0.427518)
+      (xy 1.18577 -0.77167) (xy 0.546531 -0.888112) (xy 0.085934 -0.905919) (xy -0.120962 -1.01742)
+      (xy -0.175638 -1.309737) (xy -0.177622 -1.50979) (xy -0.207161 -1.927375) (xy -0.358044 -2.098654)
+      (xy -0.716064 -2.131468) (xy -1.124338 -2.062266) (xy -1.344086 -1.898025) (xy -1.376182 -1.632916)
+      (xy -1.393515 -1.096613) (xy -1.39459 -0.372919) (xy -1.382917 0.277849) (xy -1.371614 0.71049)
+      (xy -0.177622 0.71049) (xy -0.146234 0.333156) (xy 0.021634 0.199687) (xy 0.399651 0.210774)
+      (xy 0.804605 0.29644) (xy 0.960029 0.504742) (xy 0.976924 0.71049) (xy 0.916316 1.027837)
+      (xy 0.665005 1.171624) (xy 0.399651 1.210205) (xy 0.004294 1.218127) (xy -0.151261 1.071626)
+      (xy -0.177622 0.71049) (xy -1.371614 0.71049) (xy -1.332167 2.22028) (xy -0.192326 2.273932)
+      (xy 0.490569 2.271668)) (layer B.SilkS) (width 0.01))
+    (fp_poly (pts (xy 4.174126 -0.976923) (xy 5.11751 -1.030988) (xy 5.66234 -1.073326) (xy 5.935383 -1.152422)
+      (xy 6.019852 -1.318203) (xy 6.005622 -1.563855) (xy 5.964036 -1.798983) (xy 5.856558 -1.944052)
+      (xy 5.6091 -2.024902) (xy 5.147577 -2.067373) (xy 4.484966 -2.094246) (xy 3.019581 -2.145835)
+      (xy 3.019581 2.309091) (xy 4.071984 2.309091) (xy 4.174126 -0.976923)) (layer B.SilkS) (width 0.01))
   )
   (module ao_tht:1dots (layer B.Cu)
@@
       (xy 2.828971 0.57375) (xy 3.177675 0.684638) (xy 3.240814 0.678541)) (layer B.SilkS) (width 0.01))
   )
-  (module ao_tht:1pl (layer B.Cu)
-    (at 213.5 92.4 180)
-    (fp_text reference G*** (at 0 0) (layer B.SilkS) hide
-      (effects (font (size 1.524 1.524) (thickness 0.3)) (justify mirror))
-    )
-    (fp_text value LOGO (at 0.75 0) (layer B.SilkS) hide
-      (effects (font (size 1.524 1.524) (thickness 0.3)) (justify mirror))
-    )
-    (fp_poly (pts (xy -3.286014 -2.042658) (xy -3.863287 -2.098317) (xy -4.440559 -2.153977) (xy -4.440559 -0.467664)
-      (xy -4.445178 0.315807) (xy -4.469539 0.812796) (xy -4.529405 1.092042) (xy -4.640535 1.222284)
-      (xy -4.81869 1.272262) (xy -4.84021 1.275408) (xy -5.157158 1.429016) (xy -5.23986 1.776223)
-      (xy -5.214501 2.030544) (xy -5.080468 2.162966) (xy -4.750831 2.213005) (xy -4.262937 2.220279)
-      (xy -3.286014 2.220279) (xy -3.286014 -2.042658)) (layer B.SilkS) (width 0.01))
-    (fp_poly (pts (xy -0.003238 2.234209) (xy 0.736365 2.020807) (xy 1.203103 1.685747) (xy 1.310643 1.501832)
-      (xy 1.419874 0.892083) (xy 1.357953 0.232027) (xy 1.144419 -0.298445) (xy 1.11014 -0.344105)
-      (xy 0.624368 -0.675047) (xy -0.088811 -0.853478) (xy -0.616698 -0.944735) (xy -0.88798 -1.071268)
-      (xy -0.999397 -1.305029) (xy -1.032582 -1.55543) (xy -1.113482 -1.955353) (xy -1.321451 -2.11017)
-      (xy -1.609855 -2.131469) (xy -2.131468 -2.131469) (xy -2.131468 0.710489) (xy -1.065734 0.710489)
-      (xy -1.034346 0.333156) (xy -0.866479 0.199687) (xy -0.488461 0.210774) (xy -0.083507 0.29644)
-      (xy 0.071917 0.504742) (xy 0.088811 0.710489) (xy 0.028204 1.027836) (xy -0.223107 1.171624)
-      (xy -0.488461 1.210205) (xy -0.883818 1.218127) (xy -1.039373 1.071625) (xy -1.065734 0.710489)
-      (xy -2.131468 0.710489) (xy -2.131468 2.309091) (xy -0.968102 2.309091) (xy -0.003238 2.234209)) (layer B.SilkS) (width 0.01))
-    (fp_poly (pts (xy 2.708741 2.275939) (xy 3.286014 2.220279) (xy 3.388156 -1.065735) (xy 4.269603 -1.065735)
-      (xy 4.792827 -1.077617) (xy 5.05282 -1.150333) (xy 5.141556 -1.339485) (xy 5.151049 -1.598602)
-      (xy 5.151049 -2.131469) (xy 2.131469 -2.131469) (xy 2.131469 2.331598) (xy 2.708741 2.275939)) (layer B.SilkS) (width 0.01))
-  )
   (module ao_tht:2sq (layer B.Cu)
-    (at 214.5 126.5 180)
+    (at 214.2 92.5 180)
     (fp_text reference G*** (at 0 0) (layer B.SilkS) hide
       (effects (font (size 1.524 1.524) (thickness 0.3)) (justify mirror))
@@
     (pad 1 thru_hole circle (at 0 0) (size 14 14) (drill 10) (layers *.Cu *.Mask))
   )
+  (gr_text "JLCJLCJLCJLC\n" (at 221.7 203.7) (layer F.SilkS)
+    (effects (font (size 1 1) (thickness 0.15)))
+  )
   (gr_line (start 207.5 5.6) (end 207.5 205.6) (layer Edge.Cuts) (width 0.12))
   (gr_line (start 257.5 5.6) (end 207.5 5.6) (layer Edge.Cuts) (width 0.12))
   (gr_line (start 257.5 205.6) (end 257.5 5.6) (layer Edge.Cuts) (width 0.12))
   (gr_line (start 207.5 205.6) (end 257.5 205.6) (layer Edge.Cuts) (width 0.12))
+  (zone (net 0) (net_name "") (layer F.Cu) (hatch edge 0.508)
+    (connect_pads (clearance 0.508))
+    (min_thickness 0.254)
+    (fill yes (arc_segments 32) (thermal_gap 0.508) (thermal_bridge_width 0.508))
+    (polygon
+      (pts
+        (xy 256.5 205.3) (xy 208.4 205.3) (xy 208.4 6.4) (xy 256.5 6.4)
+      )
+    )
+  )
+  (zone (net 0) (net_name "") (layer B.Cu) (hatch edge 0.508)
+    (connect_pads (clearance 0.508))
+    (min_thickness 0.254)
+    (fill yes (arc_segments 32) (thermal_gap 0.508) (thermal_bridge_width 0.508))
+    (polygon
+      (pts
+        (xy 256.5 205.3) (xy 208.4 205.3) (xy 208.4 6.4) (xy 256.5 6.4)
+      )
+    )
+  )
 )

Commit message: blah
Connections:
- REF** pad 1: (no net) -> GND (x12)
