File: kross/kross.sch (KiCad schematic (older format))
At the start: 38 parts, among them J1 CV, J2 OSC1, J3 OSC2, J4 OUT, J5 Synth_power_2x5, U1 LM13700, U2 TL072

Commit message: envy
Parts:
- R1, R10, R11, R12, R13, R14, R15, R16, R17, R2, R3, R4, R5, R6, R7, R8, R9: footprint ao_tht:R_Axial_DIN0207_L6.3mm_D2.5mm_P10.16mm_Horizontal -> ao_tht:R_Axial_DIN0207_L6.3mm_D2.5mm_P7.62mm_Horizontal
Changed lines of the file:
@@
 F 0 "R3" V 1957 1500 50  0000 C CNN
 F 1 "100K" V 1866 1500 50  0000 C CNN
-F 2 "ao_tht:R_Axial_DIN0207_L6.3mm_D2.5mm_P10.16mm_Horizontal" V 1680 1500 50  0001 C CNN
+F 2 "ao_tht:R_Axial_DIN0207_L6.3mm_D2.5mm_P7.62mm_Horizontal" V 1680 1500 50  0001 C CNN
 F 3 "" H 1750 1500 50  0001 C CNN
 F 4 "Tayda" H 1750 1500 50  0001 C CNN "Vendor"
@@
 F 0 "R4" V 1957 2150 50  0000 C CNN
 F 1 "330K" V 1866 2150 50  0000 C CNN
-F 2 "ao_tht:R_Axial_DIN0207_L6.3mm_D2.5mm_P10.16mm_Horizontal" V 1680 2150 50  0001 C CNN
+F 2 "ao_tht:R_Axial_DIN0207_L6.3mm_D2.5mm_P7.62mm_Horizontal" V 1680 2150 50  0001 C CNN
 F 3 "" H 1750 2150 50  0001 C CNN
 F 4 "Tayda" H 1750 2150 50  0001 C CNN "Vendor"
@@
 F 0 "R9" V 2607 1700 50  0000 C CNN
 F 1 "330K" V 2516 1700 50  0000 C CNN
-F 2 "ao_tht:R_Axial_DIN0207_L6.3mm_D2.5mm_P10.16mm_Horizontal" V 2330 1700 50  0001 C CNN
+F 2 "ao_tht:R_Axial_DIN0207_L6.3mm_D2.5mm_P7.62mm_Horizontal" V 2330 1700 50  0001 C CNN
 F 3 "" H 2400 1700 50  0001 C CNN
 F 4 "Tayda" H 2400 1700 50  0001 C CNN "Vendor"
@@
 F 0 "R10" V 3157 1700 50  0000 C CNN
 F 1 "100K" V 3066 1700 50  0000 C CNN
-F 2 "ao_tht:R_Axial_DIN0207_L6.3mm_D2.5mm_P10.16mm_Horizontal" V 2880 1700 50  0001 C CNN
+F 2 "ao_tht:R_Axial_DIN0207_L6.3mm_D2.5mm_P7.62mm_Horizontal" V 2880 1700 50  0001 C CNN
 F 3 "" H 2950 1700 50  0001 C CNN
 F 4 "Tayda" H 2950 1700 50  0001 C CNN "Vendor"
@@
 F 0 "R13" V 3807 1700 50  0000 C CNN
 F 1 "100K" V 3716 1700 50  0000 C CNN
-F 2 "ao_tht:R_Axial_DIN0207_L6.3mm_D2.5mm_P10.16mm_Horizontal" V 3530 1700 50  0001 C CNN
+F 2 "ao_tht:R_Axial_DIN0207_L6.3mm_D2.5mm_P7.62mm_Horizontal" V 3530 1700 50  0001 C CNN
 F 3 "" H 3600 1700 50  0001 C CNN
 F 4 "Tayda" H 3600 1700 50  0001 C CNN "Vendor"
@@
 F 0 "R1" V 1757 3850 50  0000 C CNN
 F 1 "100K" V 1666 3850 50  0000 C CNN
-F 2 "ao_tht:R_Axial_DIN0207_L6.3mm_D2.5mm_P10.16mm_Horizontal" V 1480 3850 50  0001 C CNN
+F 2 "ao_tht:R_Axial_DIN0207_L6.3mm_D2.5mm_P7.62mm_Horizontal" V 1480 3850 50  0001 C CNN
 F 3 "" H 1550 3850 50  0001 C CNN
 F 4 "Tayda" H 1550 3850 50  0001 C CNN "Vendor"
@@
 F 0 "R2" V 1757 4750 50  0000 C CNN
 F 1 "100K" V 1666 4750 50  0000 C CNN
-F 2 "ao_tht:R_Axial_DIN0207_L6.3mm_D2.5mm_P10.16mm_Horizontal" V 1480 4750 50  0001 C CNN
+F 2 "ao_tht:R_Axial_DIN0207_L6.3mm_D2.5mm_P7.62mm_Horizontal" V 1480 4750 50  0001 C CNN
 F 3 "" H 1550 4750 50  0001 C CNN
 F 4 "Tayda" H 1550 4750 50  0001 C CNN "Vendor"
@@
 F 0 "R17" V 5257 4300 50  0000 C CNN
 F 1 "1K" V 5166 4300 50  0000 C CNN
-F 2 "ao_tht:R_Axial_DIN0207_L6.3mm_D2.5mm_P10.16mm_Horizontal" V 4980 4300 50  0001 C CNN
+F 2 "ao_tht:R_Axial_DIN0207_L6.3mm_D2.5mm_P7.62mm_Horizontal" V 4980 4300 50  0001 C CNN
 F 3 "" H 5050 4300 50  0001 C CNN
 F 4 "Tayda" H 5050 4300 50  0001 C CNN "Vendor"
@@
 F 0 "R6" H 1730 4204 50  0000 R CNN
 F 1 "510R" H 1730 4295 50  0000 R CNN
-F 2 "ao_tht:R_Axial_DIN0207_L6.3mm_D2.5mm_P10.16mm_Horizontal" V 1730 4250 50  0001 C CNN
+F 2 "ao_tht:R_Axial_DIN0207_L6.3mm_D2.5mm_P7.62mm_Horizontal" V 1730 4250 50  0001 C CNN
 F 3 "" H 1800 4250 50  0001 C CNN
 F 4 "Tayda" H 1800 4250 50  0001 C CNN "Vendor"
@@
 F 0 "R7" H 1980 4204 50  0000 R CNN
 F 1 "510R" H 1980 4295 50  0000 R CNN
-F 2 "ao_tht:R_Axial_DIN0207_L6.3mm_D2.5mm_P10.16mm_Horizontal" V 1980 4250 50  0001 C CNN
+F 2 "ao_tht:R_Axial_DIN0207_L6.3mm_D2.5mm_P7.62mm_Horizontal" V 1980 4250 50  0001 C CNN
 F 3 "" H 2050 4250 50  0001 C CNN
 F 4 "Tayda" H 2050 4250 50  0001 C CNN "Vendor"
@@
 F 0 "R8" H 1980 5104 50  0000 R CNN
 F 1 "510R" H 1980 5195 50  0000 R CNN
-F 2 "ao_tht:R_Axial_DIN0207_L6.3mm_D2.5mm_P10.16mm_Horizontal" V 1980 5150 50  0001 C CNN
+F 2 "ao_tht:R_Axial_DIN0207_L6.3mm_D2.5mm_P7.62mm_Horizontal" V 1980 5150 50  0001 C CNN
 F 3 "" H 2050 5150 50  0001 C CNN
 F 4 "Tayda" H 2050 5150 50  0001 C CNN "Vendor"
@@
 F 0 "R5" H 1680 5104 50  0000 R CNN
 F 1 "510R" H 1680 5195 50  0000 R CNN
-F 2 "ao_tht:R_Axial_DIN0207_L6.3mm_D2.5mm_P10.16mm_Horizontal" V 1680 5150 50  0001 C CNN
+F 2 "ao_tht:R_Axial_DIN0207_L6.3mm_D2.5mm_P7.62mm_Horizontal" V 1680 5150 50  0001 C CNN
 F 3 "" H 1750 5150 50  0001 C CNN
 F 4 "Tayda" H 1750 5150 50  0001 C CNN "Vendor"
@@
 F 0 "R11" H 2880 3304 50  0000 R CNN
 F 1 "22K" H 2880 3395 50  0000 R CNN
-F 2 "ao_tht:R_Axial_DIN0207_L6.3mm_D2.5mm_P10.16mm_Horizontal" V 2880 3350 50  0001 C CNN
+F 2 "ao_tht:R_Axial_DIN0207_L6.3mm_D2.5mm_P7.62mm_Horizontal" V 2880 3350 50  0001 C CNN
 F 3 "" H 2950 3350 50  0001 C CNN
 F 4 "Tayda" H 2950 3350 50  0001 C CNN "Vendor"
@@
 F 0 "R12" H 3330 3304 50  0000 R CNN
 F 1 "22K" H 3330 3395 50  0000 R CNN
-F 2 "ao_tht:R_Axial_DIN0207_L6.3mm_D2.5mm_P10.16mm_Horizontal" V 3330 3350 50  0001 C CNN
+F 2 "ao_tht:R_Axial_DIN0207_L6.3mm_D2.5mm_P7.62mm_Horizontal" V 3330 3350 50  0001 C CNN
 F 3 "" H 3400 3350 50  0001 C CNN
 F 4 "Tayda" H 3400 3350 50  0001 C CNN "Vendor"
@@
 F 0 "R14" H 3730 3804 50  0000 R CNN
 F 1 "100K" H 3730 3895 50  0000 R CNN
-F 2 "ao_tht:R_Axial_DIN0207_L6.3mm_D2.5mm_P10.16mm_Horizontal" V 3730 3850 50  0001 C CNN
+F 2 "ao_tht:R_Axial_DIN0207_L6.3mm_D2.5mm_P7.62mm_Horizontal" V 3730 3850 50  0001 C CNN
 F 3 "" H 3800 3850 50  0001 C CNN
 F 4 "Tayda" H 3800 3850 50  0001 C CNN "Vendor"
@@
 F 0 "R15" H 3730 4354 50  0000 R CNN
 F 1 "15K" H 3730 4445 50  0000 R CNN
-F 2 "ao_tht:R_Axial_DIN0207_L6.3mm_D2.5mm_P10.16mm_Horizontal" V 3730 4400 50  0001 C CNN
+F 2 "ao_tht:R_Axial_DIN0207_L6.3mm_D2.5mm_P7.62mm_Horizontal" V 3730 4400 50  0001 C CNN
 F 3 "" H 3800 4400 50  0001 C CNN
 F 4 "Tayda" H 3800 4400 50  0001 C CNN "Vendor"
@@
 F 0 "R16" H 4580 4404 50  0000 R CNN
 F 1 "3.3K" H 4580 4495 50  0000 R CNN
-F 2 "ao_tht:R_Axial_DIN0207_L6.3mm_D2.5mm_P10.16mm_Horizontal" V 4580 4450 50  0001 C CNN
+F 2 "ao_tht:R_Axial_DIN0207_L6.3mm_D2.5mm_P7.62mm_Horizontal" V 4580 4450 50  0001 C CNN
 F 3 "" H 4650 4450 50  0001 C CNN
 F 4 "Tayda" H 4650 4450 50  0001 C CNN "Vendor"
