File: kross/kross.kicad_pcb (KiCad board)
At the start: 2 copper layers, 100 x 200 mm, 38 parts, among them J5 Synth_power_2x5

Commit message: more
Parts:
- removed H1: MountingHole, ao_tht:MountingHole_3.2mm_M3
- added REF**: Kosmo_Pot_Hole, ao_panel:Kosmo_Pot_Hole, F.Cu at (112.5, 88.6)
- added REF**: Kosmo_Pot_Hole, ao_panel:Kosmo_Pot_Hole, F.Cu at (112.5, 56.5)
- added REF**: Kosmo_Panel_Dual_Mounting_Holes, ao_panel:Kosmo_Panel_Dual_Mounting_Holes, F.Cu at (122.6, 217.0)
- added REF**: Kosmo_Panel_Dual_Mounting_Holes, ao_panel:Kosmo_Panel_Dual_Mounting_Holes, F.Cu at (102.5, 217.0)
- added REF**: Kosmo_Jack_Hole, ao_panel:Kosmo_Jack_Hole, F.Cu at (112.4, 157.0)
- added REF**: Kosmo_Jack_Hole, ao_panel:Kosmo_Jack_Hole, F.Cu at (112.4, 171.7)
- added REF**: Kosmo_Jack_Hole, ao_panel:Kosmo_Jack_Hole, F.Cu at (112.4, 186.5)
- added REF**: Kosmo_Jack_Hole, ao_panel:Kosmo_Jack_Hole, F.Cu at (112.4, 201.0)
Routing:
- net GND: track 158.3 -> 196.6 mm
- net Net-(C2-Pad2): track 0.00 -> 16.7 mm
- net Net-(R16-Pad2): track 74.6 -> 78.2 mm
- net Net-(R8-Pad2): track 10.8 -> 8.96 mm
Other:
- board text added: "KROSS formerly XIM @noisereap // @BlackDeath"

Commit message: sub work
Parts:
- removed the REF** at (112.4, 157.0)
- removed the REF** at (112.4, 171.7)
- added REF**: Kosmo_Jack_Hole, ao_panel:Kosmo_Jack_Hole, F.Cu at (112.2, 157.6)
- added REF**: Kosmo_Jack_Hole, ao_panel:Kosmo_Jack_Hole, F.Cu at (112.3, 172.0)
- moved C1 47.4 mm to (91.4, 44.5)
- moved C2 47.4 mm to (75.4, 44.5)
- moved C3 47.4 mm to (89.4, 70.7)
- moved CV 47.4 mm to (86.4, 144.5)
- moved CVATTN1 47.4 mm to (84.4, 88.5)
- moved D3 47.4 mm to (87.9, 49.0)
- moved D4 47.4 mm to (80.9, 41.5)
- moved J5 47.4 mm to (79.4, 36.5)
- moved MIX1 47.4 mm to (84.4, 56.5)
- moved OSC1 47.4 mm to (74.4, 144.5)
- moved OSC1 47.4 mm to (80.4, 144.5)
- moved OUT 47.4 mm to (91.9, 144.5)
- moved R10 47.4 mm to (93.2, 123.8)
- moved R12 47.4 mm to (93.9, 106.0)
- moved R14 47.4 mm to (84.2, 126.6)
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Routing:
- net GND: track 196.6 -> 196.1 mm
Other:
- board size 100 x 200 mm -> 52.6 x 200 mm

Commit message: envy
Parts:
- removed LM13700: LM13700, ao_tht:DIP-16_W7.62mm_Socket_LongPads
- removed the OSC1 at (74.4, 144.5)
- removed the OSC1 at (80.4, 144.5)
- removed the REF** at (112.2, 157.6)
- removed the REF** at (112.3, 172.0)
- removed the REF** at (112.4, 186.5)
- removed TL072: TL072, ao_tht:DIP-8_W7.62mm_Socket_LongPads
- added G***: LOGO, ao_tht:cross, B.Cu at (80.5, 47.5)
- added G***: LOGO, ao_tht:cross, B.Cu at (112.5, 117.5)
- added G***: LOGO, ao_tht:o, B.Cu at (103.0, 194.0)
- added G***: LOGO, ao_tht:x, B.Cu at (102.5, 177.0)
- added G***: LOGO, ao_tht:2, B.Cu at (102.5, 158.5)
- added G***: LOGO, ao_tht:1, B.Cu at (102.5, 140.5)
- added G***: LOGO, ao_tht:BD3, F.Cu at (112.5, 113.5)
- added G***: LOGO, ao_tht:kross, B.Cu at (112.5, 37.0)
- added H1: MountingHole, ao_tht:MountingHole_3.2mm_M3, F.Cu at (181.0, 184.0)
- added OSC1: OSC1, ao_tht:Molex_KK-254_AE-6410-02A_1x02_P2.54mm_Vertical, F.Cu at (69.8, 133.0)
- added OSC2: OSC2, ao_tht:Molex_KK-254_AE-6410-02A_1x02_P2.54mm_Vertical, F.Cu at (76.2, 133.0)
- added REF**: Kosmo_Jack_Hole, ao_panel:Kosmo_Jack_Hole, F.Cu at (112.5, 147.0)
- added REF**: Kosmo_Jack_Hole, ao_panel:Kosmo_Jack_Hole, F.Cu at (112.5, 165.0)
- added REF**: Kosmo_Jack_Hole, ao_panel:Kosmo_Jack_Hole, F.Cu at (112.4, 183.0)
- added U1: LM13700, ao_tht:DIP-16_W7.62mm_Socket_LongPads, F.Cu at (88.6, 99.2)
- added U2: TL072, ao_tht:DIP-8_W7.62mm_Socket_LongPads, F.Cu at (81.8, 70.4)
- R1, R10, R11, R12, R13, R14, R15, R16, R17, R2, R3, R4, R5, R6, R7, R8, R9: footprint ao_tht:R_Axial_DIN0207_L6.3mm_D2.5mm_P10.16mm_Horizontal -> ao_tht:R_Axial_DIN0207_L6.3mm_D2.5mm_P7.62mm_Horizontal
- moved CV 12.2 mm to (82.2, 133.0)
- moved OUT 12.2 mm to (87.7, 133.0)
- moved H2 11.1 mm to (70.5, 55.0)
- moved R2 10.6 mm to (73.6, 127.2)
- moved R1 10.6 mm to (70.5, 127.2)
- moved R15 10.6 mm to (76.5, 127.2)
- moved R6 10.6 mm to (82.7, 127.2)
- moved R17 8.51 mm to (88.6, 119.5)
- moved R14 8.38 mm to (79.6, 119.6)
- moved R10 7.74 mm to (89.0, 117.3)
- moved R7 7.74 mm to (70.5, 117.3)
- moved R8 7.74 mm to (73.7, 117.3)
- moved C1 6.02 mm to (86.9, 48.5)
- moved C2 6.02 mm to (70.9, 48.5)
- moved D3 6.02 mm to (83.4, 53.0)
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Routing:
- net Net-(D1-Pad2): track 216.3 -> 74.4 mm
- net Net-(MIX1-Pad2): track 86.6 -> 16.2 mm
- net Net-(C2-Pad2): track 16.7 -> 86.7 mm
- net Net-(R2-Pad2): track 66.9 -> 17.4 mm
- net Net-(R10-Pad2): track 80.5 -> 50.6 mm, vias 0 -> 1
- net Net-(CVATTN1-Pad1): track 118.8 -> 102.8 mm
- net GND: track 196.1 -> 181.2 mm
- net Net-(R7-Pad2): track 16.5 -> 25.9 mm
- net Net-(CVATTN1-Pad3): track 50.4 -> 42.5 mm
- net Net-(C1-Pad1): track 83.0 -> 77.5 mm
- net Net-(R3-Pad2): track 63.0 -> 58.0 mm
- net Net-(R14-Pad1): track 33.9 -> 30.3 mm
- net Net-(D2-Pad2): track 30.5 -> 27.7 mm
- net Net-(D2-Pad1): track 3.51 -> 6.05 mm
- net Net-(J4-Pad1): track 8.32 -> 6.25 mm
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- added copper zone on B.Cu, net (none)
- added copper zone on F.Cu, net (none)
- removed copper zone on F.Cu, net GND
- removed copper zone on B.Cu, net Net-(C2-Pad2)
Other:
- board size 52.6 x 200 mm -> 57.1 x 200 mm
- board text added: "JLCJLCJLCJLC"
- board text added: "designed in Bergen, Norway"

Commit message: blah
Parts:
- removed H1: MountingHole, ao_tht:MountingHole_3.2mm_M3
- moved REF** 0.40 mm to (122.2, 217.0)
- moved REF** 0.30 mm to (102.8, 217.0)
Connections:
- REF** pad 1: (no net) -> GND (x8)
Routing:
- added copper zone on B.Cu, net GND
- added copper zone on F.Cu, net GND
