File: envy/envy.kicad_pcb (KiCad board)
At the start: 2 copper layers, 57.1 x 200 mm, 42 parts, among them J1 CV, J2 OUT, J3 INVOUT, J5 Synth_power_2x5, U1 TL074

Commit message: more envy
Parts:
- removed the G*** at (112.1, 37.7)
- added G***: LOGO, ao_tht:envy5, B.Cu at (70.5, 114.9)
- added G***: LOGO, ao_tht:envy5, B.Cu at (111.9, 39.2)
- added G***: LOGO, ao_tht:pipe, B.Cu at (102.8, 115.8)
- added G***: LOGO, ao_tht:slash_right, B.Cu at (103.4, 86.6)
- added G***: LOGO, ao_tht:slash_left, B.Cu at (103.2, 55.0)
- moved G*** 15.6 mm to (121.4, 60.0)
- moved REF** 0.80 mm to (112.5, 121.1)
- moved RV3 0.75 mm to (80.2, 121.0)
- moved REF** 0.40 mm to (112.5, 106.8)
- moved D1 0.30 mm to (81.5, 106.8)
- moved R9 0.20 mm to (78.0, 70.3)
- moved REF** 0.20 mm to (122.4, 217.0)
- renumbered J1 to IN, J3 to INV
Routing:
- net GND: track 41.1 -> 125.7 mm
- net Net-(R2-Pad1): track 0.00 -> 67.2 mm
- net Net-(R9-Pad2): track 0.00 -> 63.0 mm
- net Net-(C5-Pad2): track 0.00 -> 49.0 mm
- net Net-(D2-Pad2): track 0.00 -> 47.0 mm
- net Net-(D1-Pad1): track 0.00 -> 46.4 mm
- net Net-(C2-Pad2): track 6.07 -> 49.1 mm
- net Net-(RV1-Pad1): track 0.00 -> 37.3 mm
- net Net-(J3-Pad1): track 0.00 -> 30.5 mm
- net Net-(C5-Pad1): track 0.00 -> 26.8 mm
- net Net-(R6-Pad2): track 0.00 -> 26.5 mm
- net Net-(C1-Pad1): track 5.95 -> 32.2 mm
- net Net-(J2-Pad1): track 0.00 -> 22.1 mm
- net Net-(D2-Pad1): track 0.00 -> 21.4 mm
- net Net-(R5-Pad2): track 0.00 -> 18.5 mm
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- added copper zone on B.Cu, net GND
Other:
- board text added: "ENVY v0.1 @BlackDeath Bumm Bumm Garage 2021"
- board text added: "Sound in! Voltage out!"
- board text added: "designed in Bergen, Norway"
