File: xorcist/xorcist/xorcist.kicad_pcb (KiCad board)
At the start: 2 copper layers, 108 x 200 mm, 73 parts, among them J1 Synth_power_2x5, Q1 2N3904, SW1 SW_SPDT, SW2 SW_SPDT, U1 40106, U2 TL074, U3 4070

Commit message: add springy
Parts:
- added G***: LOGO, ao_tht:BD3, B.Cu at (314.0, 149.2)
- added G***: LOGO, ao_tht:cross, B.Cu at (384.8, 107.8)
- moved REF** 0.25 mm to (384.8, 133.0)
- moved REF** 0.25 mm to (361.0, 133.0)
