File: niga/niga/niga.sch (KiCad schematic (older format))
At the start: 11 parts

Commit message: finalize xorcist spring niga
Parts:
- added C1, C2: 10uf, ao_tht:CP_Radial_D6.3mm_P2.50mm, symbol ao_tht:CP
- added C3, C4: 100nf, ao_tht:C_Disc_D3.0mm_W1.6mm_P2.50mm, symbol ao_tht:C
- added D1, D2: 1N4148, ao_tht:D_DO-35_SOD27_P7.62mm_Horizontal, symbol Device:D
- added J3: Synth_power_2x5, ao_tht:Power_Header, symbol ao_tht:Synth_power_2x5
- added unit 3 of U1
- J1, J2: renamed from J?; footprint (none) -> ao_tht:Molex_KK-254_AE-6410-02A_1x02_P2.54mm_Vertical
- RV1, RV2, RV3: renamed from RV?; footprint (none) -> ao_tht:Molex_KK-254_AE-6410-03A_1x03_P2.54mm_Vertical
- U1: renamed from U?; footprint (none) -> ao_tht:DIP-8_W7.62mm_Socket_LongPads
- gave numbers to parts that had none: 4
Connections:
- net GND: now also J1.2 (Pin_2), C1.2, C2.1, C3.1, C4.2, J3.3 (GND), J3.4 (GND), J3.5 (GND), J3.6 (GND), J3.7 (GND), J3.8 (GND)
- net at R3.1: now also U1.5 (+); no longer U1.3 (+)
- new net: R4.2, U1.6 (-), U1.7
- new net: C1.1, C3.2, D1.1 (K), U1.8 (V+)
- new net: D1.2 (A), J3.10 (+12V), J3.9 (+12V)
- new net: C2.2, C4.1, D2.2 (A), U1.4 (V-)
- new net: D2.1 (K), J3.1 (-12V), J3.2 (-12V)
